File: hardware/rcj25.kicad_sch (KiCad schematic)
At the start: 39 parts, among them J2 USB_B_Micro, J3 Conn_01x12_Pin, J4 Conn_01x24_MountingPin, SW2 SW_Push_Shielded, U1 RP2040, U2 LIS3DH, U3 W25X40CLSV, U4 LM1117MP-ADJ, U5 AP7365, Y1 Crystal_GND24

Commit message: she go brrr
Parts:
- C14: value C -> 1u
Changed lines of the file:
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@@
 			)
 		)
-		(property "Value" "C"
+		(property "Value" "1u"
 			(at 148.59 92.7099 0)
 			(effects
