File: hardware/rcj25.kicad_pcb (KiCad board)
At the start: 2 copper layers, 26.5 x 26.8 mm, 39 parts, among them J2 USB_B_Micro, J3 Conn_01x12_Pin, J4 Conn_01x24_MountingPin, SW2 SW_Push_Shielded, U1 RP2040, U2 LIS3DH, U3 W25X40CLSV, U4 LM1117MP-ADJ, U5 AP7365, Y1 Crystal_GND24

Commit message: she go brrr
Routing:
- net Net-(U1-GPIO26_ADC0): track 20.0 -> 19.3 mm
Changed lines of the file:
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@@
 	)
 	(segment
-		(start 107.5875 55.1625)
-		(end 107.925 55.1625)
-		(width 0.2)
-		(layer "F.Cu")
-		(net 2)
-	)
-	(segment
 		(start 112.44 56.41)
 		(end 112.44 54.925)
@@
 	)
 	(segment
-		(start 108.1625 54.925)
-		(end 112.44 54.925)
+		(start 111.9 59.8)
+		(end 112.19038 59.50962)
 		(width 0.2)
 		(layer "F.Cu")
@@
 	)
 	(segment
-		(start 111.9 59.8)
-		(end 112.19038 59.50962)
+		(start 115.515 60.625)
+		(end 114.39962 59.50962)
 		(width 0.2)
 		(layer "F.Cu")
@@
 	)
 	(segment
-		(start 115.515 60.625)
-		(end 114.39962 59.50962)
+		(start 106.25 56.8375)
+		(end 107.925 55.1625)
+		(width 0.2)
+		(layer "F.Cu")
+		(net 2)
+	)
+	(segment
+		(start 112.2025 55.1625)
+		(end 112.44 54.925)
 		(width 0.2)
 		(layer "F.Cu")
@@
 	)
 	(segment
-		(start 106.25 56.5)
-		(end 107.5875 55.1625)
-		(width 0.2)
-		(layer "F.Cu")
-		(net 2)
-	)
-	(segment
 		(start 99.974 68.150848)
 		(end 99.974 67.649152)
@@
 	)
 	(segment
-		(start 107.925 55.1625)
-		(end 108.1625 54.925)
-		(width 0.2)
-		(layer "F.Cu")
-		(net 2)
-	)
-	(segment
-		(start 106.25 57.5)
-		(end 106.25 56.5)
+		(start 98.9 61.65)
+		(end 98.9 63.325)
 		(width 0.2)
 		(layer "F.Cu")
@@
 	)
 	(segment
-		(start 98.9 61.65)
-		(end 98.9 63.325)
+		(start 100.55 68.4)
+		(end 100.223152 68.4)
 		(width 0.2)
 		(layer "F.Cu")
@@
 	)
 	(segment
-		(start 100.55 68.4)
-		(end 100.223152 68.4)
+		(start 106.25 57.5)
+		(end 106.25 56.8375)
 		(width 0.2)
 		(layer "F.Cu")
@@
 	)
 	(segment
+		(start 107.925 55.1625)
+		(end 112.2025 55.1625)
+		(width 0.2)
+		(layer "F.Cu")
+		(net 2)
+	)
+	(segment
 		(start 98.1 68.9)
 		(end 97.55 69.45)
@@
 	)
 	(segment
+		(start 108.3 74.5)
+		(end 108.3 72.144314)
+		(width 0.2)
+		(layer "F.Cu")
+		(net 3)
+	)
+	(segment
 		(start 110.7625 68.2625)
 		(end 110.8875 68.1375)
@@
 	)
 	(segment
-		(start 98.4 75.3)
-		(end 107.5 75.3)
+		(start 96.825 66.85)
+		(end 96.05 67.625)
 		(width 0.2)
 		(layer "F.Cu")
@@
 	)
 	(segment
-		(start 107.5 75.3)
-		(end 108.3 74.5)
-		(width 0.2)
-		(layer "F.Cu")
-		(net 3)
-	)
-	(segment
-		(start 96.05 72.95)
-		(end 98.4 75.3)
-		(width 0.2)
-		(layer "F.Cu")
-		(net 3)
-	)
-	(segment
 		(start 110.9 70.425)
 		(end 109.4 70.425)
@@
 	)
 	(segment
+		(start 96.05 67.625)
+		(end 96.05 72.95)
+		(width 0.2)
+		(layer "F.Cu")
+		(net 3)
+	)
+	(segment
 		(start 109.8635 63.6865)
 		(end 110.195577 63.354423)
@@
 	)
 	(segment
-		(start 108.3 74.5)
-		(end 108.3 72.144314)
-		(width 0.2)
-		(layer "F.Cu")
-		(net 3)
-	)
-	(segment
 		(start 114.425 56.25)
 		(end 113.8 56.25)
@@
 	)
 	(segment
-		(start 96.825 66.85)
-		(end 96.05 67.625)
-		(width 0.2)
-		(layer "F.Cu")
-		(net 3)
-	)
-	(segment
 		(start 114.425 56.25)
 		(end 113.85 56.25)
@@
 	)
 	(segment
-		(start 96.05 67.625)
-		(end 96.05 72.95)
-		(width 0.2)
-		(layer "F.Cu")
-		(net 3)
-	)
-	(segment
 		(start 104.587503 65.7375)
 		(end 105.222578 66.372575)
@@
 	)
 	(segment
+		(start 98.4 75.3)
+		(end 107.5 75.3)
+		(width 0.2)
+		(layer "F.Cu")
+		(net 3)
+	)
+	(segment
+		(start 107.5 75.3)
+		(end 108.3 74.5)
+		(width 0.2)
+		(layer "F.Cu")
+		(net 3)
+	)
+	(segment
 		(start 110.05 68.975)
 		(end 110.7625 68.2625)
@@
 	)
 	(segment
+		(start 96.05 72.95)
+		(end 98.4 75.3)
+		(width 0.2)
+		(layer "F.Cu")
+		(net 3)
+	)
+	(segment
 		(start 103.209 70.941)
 		(end 103.209 71.91605)
@@
 	)
 	(segment
-		(start 100 55.4)
-		(end 97.9 57.5)
+		(start 113.3 60.1)
+		(end 113.295767 60.1)
 		(width 0.2)
 		(layer "F.Cu")
@@
 	)
 	(segment
-		(start 113.3 60.1)
-		(end 113.295767 60.1)
+		(start 100.050003 55.4)
+		(end 100 55.4)
 		(width 0.2)
 		(layer "F.Cu")
@@
 	)
 	(segment
-		(start 100 55.25)
-		(end 100 55.4)
+		(start 100.2 55.250003)
+		(end 100.050003 55.4)
+		(width 0.2)
+		(layer "F.Cu")
+		(net 7)
+	)
+	(segment
+		(start 100 55.4)
+		(end 97.9 57.5)
 		(width 0.2)
 		(layer "F.Cu")
@@
 	)
 	(via
-		(at 100 55.25)
+		(at 100.2 55.250003)
 		(size 0.6)
 		(drill 0.3)
@@
 	)
 	(segment
-		(start 94.7 61.2)
-		(end 94.7 69.47)
-		(width 0.5)
-		(layer "B.Cu")
-		(net 7)
-	)
-	(segment
-		(start 112.4 55.200001)
-		(end 111.449999 54.25)
+		(start 103.7115 56.8615)
+		(end 108.476 56.8615)
 		(width 0.2)
 		(layer "B.Cu")
@@
 	)
 	(segment
-		(start 109.1875 55.8875)
-		(end 108.2135 56.8615)
-		(width 0.2)
+		(start 94.7 61.2)
+		(end 94.7 69.47)
+		(width 0.5)
 		(layer "B.Cu")
 		(net 7)
 	)
 	(segment
-		(start 100.1 55.15)
-		(end 100 55.25)
+		(start 112.4 55.200001)
+		(end 111.449999 54.25)
 		(width 0.2)
 		(layer "B.Cu")
@@
 	)
 	(segment
-		(start 108.2135 56.8615)
-		(end 103.7115 56.8615)
-		(width 0.2)
-		(layer "B.Cu")
-		(net 7)
-	)
-	(segment
 		(start 109.1875 56.15)
 		(end 111.450001 56.15)
@@
 	)
 	(segment
-		(start 102 55.15)
-		(end 100.1 55.15)
+		(start 102.100003 55.250003)
+		(end 103.7115 56.8615)
 		(width 0.2)
 		(layer "B.Cu")
@@
 	)
 	(segment
-		(start 103.7115 56.8615)
-		(end 102 55.15)
+		(start 108.476 56.8615)
+		(end 109.1875 56.15)
+		(width 0.2)
+		(layer "B.Cu")
+		(net 7)
+	)
+	(segment
+		(start 100.2 55.250003)
+		(end 102.100003 55.250003)
 		(width 0.2)
 		(layer "B.Cu")
@@
 	)
 	(segment
-		(start 98.1 68.4)
-		(end 96.95 68.4)
+		(start 103.075 68.975)
+		(end 102.522355 69.527643)
 		(width 0.2)
 		(layer "F.Cu")
@@
 	)
 	(segment
-		(start 103.075 68.975)
-		(end 102.522355 69.527643)
+		(start 98.1 68.4)
+		(end 96.95 68.4)
 		(width 0.2)
 		(layer "F.Cu")
@@
 	)
 	(segment
-		(start 113.049 57.845728)
-		(end 113.049 58.624983)
-		(width 0.2)
-		(layer "B.Cu")
-		(net 59)
-	)
-	(segment
-		(start 114.4 53.7)
-		(end 114.4 56.494728)
-		(width 0.2)
-		(layer "B.Cu")
-		(net 59)
-	)
-	(segment
-		(start 113.85 63.85)
+		(start 114.4 63.3)
 		(end 109.7 68)
 		(width 0.2)
@@
 	)
 	(segment
-		(start 113.85 59.425983)
-		(end 113.85 63.85)
-		(width 0.2)
-		(layer "B.Cu")
-		(net 59)
-	)
-	(segment
-		(start 114.4 56.494728)
-		(end 113.049 57.845728)
-		(width 0.2)
-		(layer "B.Cu")
-		(net 59)
-	)
-	(segment
-		(start 113.049 58.624983)
-		(end 113.85 59.425983)
+		(start 114.4 53.7)
+		(end 114.4 63.3)
 		(width 0.2)
 		(layer "B.Cu")
@@
 		(layers "F.Cu" "B.Cu")
 		(hatch edge 0.5)
-		(connect_pads
+		(connect_pads yes
 			(clearance 0.5)
 		)
 		(min_thickness 0.25)
 		(filled_areas_thickness no)
-		(fill yes
+		(fill
 			(thermal_gap 0.5)
 			(thermal_bridge_width 0.5)

Commit message: I see light
Parts:
- C13, C15: value C -> NC
- R7: value R -> 120
- R8: value R -> 150
Changed lines of the file:
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@@
 			)
 		)
-		(property "Value" "R"
+		(property "Value" "120"
 			(at 0 -1.43 0)
 			(layer "B.Fab")
@@
 			)
 		)
-		(property "Value" "C"
+		(property "Value" "NC"
 			(at 0 -1.43 0)
 			(layer "B.Fab")
@@
 			)
 		)
-		(property "Value" "R"
+		(property "Value" "150"
 			(at 0 -1.43 0)
 			(layer "B.Fab")
@@
 			)
 		)
-		(property "Value" "C"
+		(property "Value" "NC"
 			(at 0 -1.43 0)
 			(layer "B.Fab")
@@
 		(min_thickness 0.25)
 		(filled_areas_thickness no)
-		(fill
+		(fill yes
 			(thermal_gap 0.5)
 			(thermal_bridge_width 0.5)
